Commit message: attempting to fix simulation problem that makes fingers go crazy, and joint velocity goes nan for some reason

File: dlr_description/urdf/hit2/hit2.gazebo.xacro (robot description, xacro)
@@ -2,15 +2,31 @@
 <robot xmlns:xacro="http://www.ros.org/wiki/xacro">
     <xacro:macro name="dlr_hit2_gazebo" params="name">
+        <!-- set friction properties -->
+        <xacro:property name="gazebo_friction_properties">
+            <gravity>true</gravity>
+            <mu1>500.0</mu1>
+            <mu2>500.0</mu2>
+            <kp>1000000.0</kp>
+            <kd>100.0</kd>
+            <!-- <fdir1>string</fdir1> -->
+            <!-- <dampingFactor>double</dampingFactor> -->
+            <!-- <maxVel>double</maxVel> -->
+            <!-- <minDepth>double</minDepth> -->
+            <!-- <maxContacts>int</maxContacts> -->
+        </xacro:property>
+        <!-- <xacro:insert_block name="gazebo_friction_properties"/> -->
         <gazebo reference="${name}_palm_link">
             <material>DLR/LightGrey</material>
-            <turnGravityOff>false</turnGravityOff>
+            <!-- <turnGravityOff>false</turnGravityOff> -->
+            <xacro:insert_block name="gazebo_friction_properties"/>
         </gazebo>
         <gazebo reference="${name}_thumb_abd_link">
             <material>DLR/LightGrey</material>
-            <turnGravityOff>false</turnGravityOff>
+            <!-- <turnGravityOff>false</turnGravityOff> -->
+            <xacro:insert_block name="gazebo_friction_properties"/>
         </gazebo>
         <gazebo reference="${name}_thumb_proximal_link">
-            <selfCollide>true</selfCollide>
-            <sensor name='${name}_thumb_proximal_contact_sensor' type='contact'>
+            <!-- <selfCollide>true</selfCollide> -->
+            <!-- <sensor name='${name}_thumb_proximal_contact_sensor' type='contact'>
                 <always_on>true</always_on>
                 <update_rate>100</update_rate>
@@ -24,11 +40,12 @@
                     <bumperTopicName>${name}_finger_12_bumper</bumperTopicName>
                 </plugin>
-            </sensor>
-            <material>DLR/LightGrey</material>
-            <turnGravityOff>false</turnGravityOff>
+            </sensor> -->
+            <material>DLR/LightGrey</material>
+            <!-- <turnGravityOff>false</turnGravityOff> -->
+            <xacro:insert_block name="gazebo_friction_properties"/>
         </gazebo>
         <gazebo reference="${name}_thumb_medial_link">
-            <selfCollide>true</selfCollide>
-            <sensor name='${name}_thumb_medial_contact_sensor' type='contact'>
+            <!-- <selfCollide>true</selfCollide>  -->
+            <!-- <sensor name='${name}_thumb_medial_contact_sensor' type='contact'>
                 <always_on>true</always_on>
                 <update_rate>100</update_rate>
@@ -42,10 +59,11 @@
                     <bumperTopicName>${name}_thumb_medial_bumper</bumperTopicName>
                 </plugin>
-            </sensor>
-            <material>DLR/LightGrey</material>
+            </sensor> -->
+            <material>DLR/LightGrey</material>
+            <xacro:insert_block name="gazebo_friction_properties"/>
         </gazebo>
         <gazebo reference="${name}_thumb_distal_link">
-            <selfCollide>true</selfCollide>
-            <sensor name='${name}_thumb_distal_contact_sensor' type='contact'>
+            <!-- <selfCollide>true</selfCollide>  -->
+            <!-- <sensor name='${name}_thumb_distal_contact_sensor' type='contact'>
                 <always_on>true</always_on>
                 <update_rate>100</update_rate>
@@ -59,14 +77,16 @@
                     <bumperTopicName>${name}_thumb_distal_bumper</bumperTopicName>
                 </plugin>
-            </sensor>
-            <material>DLR/LightGrey</material>
+            </sensor> -->
+            <material>DLR/LightGrey</material>
+            <xacro:insert_block name="gazebo_friction_properties"/>
         </gazebo>
         <gazebo reference="${name}_index_abd_link">
             <material>DLR/LightGrey</material>
-            <turnGravityOff>false</turnGravityOff>
+            <!-- <turnGravityOff>false</turnGravityOff> -->
+            <xacro:insert_block name="gazebo_friction_properties"/>
         </gazebo>
         <gazebo reference="${name}_index_proximal_link">
-            <selfCollide>true</selfCollide>
-            <sensor name='${name}_index_proximal_contact_sensor' type='contact'>
+            <!-- <selfCollide>true</selfCollide> -->
+            <!-- <sensor name='${name}_index_proximal_contact_sensor' type='contact'>
                 <always_on>true</always_on>
                 <update_rate>100</update_rate>
@@ -80,11 +100,12 @@
                     <bumperTopicName>${name}_finger_12_bumper</bumperTopicName>
                 </plugin>
-            </sensor>
-            <material>DLR/LightGrey</material>
-            <turnGravityOff>false</turnGravityOff>
+            </sensor> -->
+            <material>DLR/LightGrey</material>
+            <!-- <turnGravityOff>false</turnGravityOff> -->
+            <xacro:insert_block name="gazebo_friction_properties"/>
         </gazebo>
         <gazebo reference="${name}_index_medial_link">
-            <selfCollide>true</selfCollide>
-            <sensor name='${name}_index_medial_contact_sensor' type='contact'>
+            <!-- <selfCollide>true</selfCollide>  -->
+            <!-- <sensor name='${name}_index_medial_contact_sensor' type='contact'>
                 <always_on>true</always_on>
                 <update_rate>100</update_rate>
@@ -98,10 +119,11 @@
                     <bumperTopicName>${name}_index_medial_bumper</bumperTopicName>
                 </plugin>
-            </sensor>
-            <material>DLR/LightGrey</material>
+            </sensor> -->
+            <material>DLR/LightGrey</material>
+            <xacro:insert_block name="gazebo_friction_properties"/>
         </gazebo>
         <gazebo reference="${name}_index_distal_link">
-            <selfCollide>true</selfCollide>
-            <sensor name='${name}_index_distal_contact_sensor' type='contact'>
+            <!-- <selfCollide>true</selfCollide>  -->
+            <!-- <sensor name='${name}_index_distal_contact_sensor' type='contact'>
                 <always_on>true</always_on>
                 <update_rate>100</update_rate>
@@ -115,14 +137,16 @@
                     <bumperTopicName>${name}_index_distal_bumper</bumperTopicName>
                 </plugin>
-            </sensor>
-            <material>DLR/LightGrey</material>
+            </sensor> -->
+            <material>DLR/LightGrey</material>
+            <xacro:insert_block name="gazebo_friction_properties"/>
         </gazebo>
         <gazebo reference="${name}_middle_abd_link">
             <material>DLR/LightGrey</material>
-            <turnGravityOff>false</turnGravityOff>
+            <!-- <turnGravityOff>false</turnGravityOff> -->
+            <xacro:insert_block name="gazebo_friction_properties"/>
         </gazebo>
         <gazebo reference="${name}_middle_proximal_link">
-            <selfCollide>true</selfCollide>
-            <sensor name='${name}_middle_proximal_contact_sensor' type='contact'>
+            <!-- <selfCollide>true</selfCollide> -->
+            <!-- <sensor name='${name}_middle_proximal_contact_sensor' type='contact'>
                 <always_on>true</always_on>
                 <update_rate>100</update_rate>
@@ -136,11 +160,12 @@
                     <bumperTopicName>${name}_finger_12_bumper</bumperTopicName>
                 </plugin>
-            </sensor>
-            <material>DLR/LightGrey</material>
-            <turnGravityOff>false</turnGravityOff>
+            </sensor> -->
+            <material>DLR/LightGrey</material>
+            <!-- <turnGravityOff>false</turnGravityOff> -->
+            <xacro:insert_block name="gazebo_friction_properties"/>
         </gazebo>
         <gazebo reference="${name}_middle_medial_link">
-            <selfCollide>true</selfCollide>
-            <sensor name='${name}_middle_medial_contact_sensor' type='contact'>
+            <!-- <selfCollide>true</selfCollide>  -->
+            <!-- <sensor name='${name}_middle_medial_contact_sensor' type='contact'>
                 <always_on>true</always_on>
                 <update_rate>100</update_rate>
@@ -154,10 +179,11 @@
                     <bumperTopicName>${name}_middle_medial_bumper</bumperTopicName>
                 </plugin>
-            </sensor>
-            <material>DLR/LightGrey</material>
+            </sensor> -->
+            <material>DLR/LightGrey</material>
+            <xacro:insert_block name="gazebo_friction_properties"/>
         </gazebo>
         <gazebo reference="${name}_middle_distal_link">
-            <selfCollide>true</selfCollide>
-            <sensor name='${name}_middle_distal_contact_sensor' type='contact'>
+            <!-- <selfCollide>true</selfCollide>  -->
+            <!-- <sensor name='${name}_middle_distal_contact_sensor' type='contact'>
                 <always_on>true</always_on>
                 <update_rate>100</update_rate>
@@ -171,6 +197,7 @@
                     <bumperTopicName>${name}_middle_distal_bumper</bumperTopicName>
                 </plugin>
-            </sensor>
-            <material>DLR/LightGrey</material>
+            </sensor> -->
+            <material>DLR/LightGrey</material>
+            <xacro:insert_block name="gazebo_friction_properties"/>
         </gazebo>
         <gazebo reference="${name}_ring_abd_link">
@@ -179,6 +206,6 @@
         </gazebo>
         <gazebo reference="${name}_ring_proximal_link">
-            <selfCollide>true</selfCollide>
-            <sensor name='${name}_ring_proximal_contact_sensor' type='contact'>
+            <!-- <selfCollide>true</selfCollide> -->
+            <!-- <sensor name='${name}_ring_proximal_contact_sensor' type='contact'>
                 <always_on>true</always_on>
                 <update_rate>100</update_rate>
@@ -192,11 +219,12 @@
                     <bumperTopicName>${name}_finger_12_bumper</bumperTopicName>
                 </plugin>
-            </sensor>
-            <material>DLR/LightGrey</material>
-            <turnGravityOff>false</turnGravityOff>
+            </sensor> -->
+            <material>DLR/LightGrey</material>
+            <!-- <turnGravityOff>false</turnGravityOff> -->
+            <xacro:insert_block name="gazebo_friction_properties"/>
         </gazebo>
         <gazebo reference="${name}_ring_medial_link">
-            <selfCollide>true</selfCollide>
-            <sensor name='${name}_ring_medial_contact_sensor' type='contact'>
+            <!-- <selfCollide>true</selfCollide>  -->
+            <!-- <sensor name='${name}_ring_medial_contact_sensor' type='contact'>
                 <always_on>true</always_on>
                 <update_rate>100</update_rate>
@@ -210,10 +238,11 @@
                     <bumperTopicName>${name}_ring_medial_bumper</bumperTopicName>
                 </plugin>
-            </sensor>
-            <material>DLR/LightGrey</material>
+            </sensor> -->
+            <material>DLR/LightGrey</material>
+            <xacro:insert_block name="gazebo_friction_properties"/>
         </gazebo>
         <gazebo reference="${name}_ring_distal_link">
-            <selfCollide>true</selfCollide>
-            <sensor name='${name}_ring_distal_contact_sensor' type='contact'>
+            <!-- <selfCollide>true</selfCollide>  -->
+            <!-- <sensor name='${name}_ring_distal_contact_sensor' type='contact'>
                 <always_on>true</always_on>
                 <update_rate>100</update_rate>
@@ -227,14 +256,16 @@
                     <bumperTopicName>${name}_ring_distal_bumper</bumperTopicName>
                 </plugin>
-            </sensor>
-            <material>DLR/LightGrey</material>
+            </sensor> -->
+            <material>DLR/LightGrey</material>
+            <xacro:insert_block name="gazebo_friction_properties"/>
         </gazebo>
         <gazebo reference="${name}_pinky_abd_link">
             <material>DLR/LightGrey</material>
-            <turnGravityOff>false</turnGravityOff>
+            <!-- <turnGravityOff>false</turnGravityOff> -->
+            <xacro:insert_block name="gazebo_friction_properties"/>
         </gazebo>
         <gazebo reference="${name}_pinky_proximal_link">
-            <selfCollide>true</selfCollide>
-            <sensor name='${name}_pinky_proximal_contact_sensor' type='contact'>
+            <!-- <selfCollide>true</selfCollide> -->
+            <!-- <sensor name='${name}_pinky_proximal_contact_sensor' type='contact'>
                 <always_on>true</always_on>
                 <update_rate>100</update_rate>
@@ -248,11 +279,12 @@
                     <bumperTopicName>${name}_finger_12_bumper</bumperTopicName>
                 </plugin>
-            </sensor>
-            <material>DLR/LightGrey</material>
-            <turnGravityOff>false</turnGravityOff>
+            </sensor> -->
+            <material>DLR/LightGrey</material>
+            <!-- <turnGravityOff>false</turnGravityOff> -->
+            <xacro:insert_block name="gazebo_friction_properties"/>
         </gazebo>
         <gazebo reference="${name}_pinky_medial_link">
-            <selfCollide>true</selfCollide>
-            <sensor name='${name}_pinky_medial_contact_sensor' type='contact'>
+            <!-- <selfCollide>true</selfCollide>  -->
+            <!-- <sensor name='${name}_pinky_medial_contact_sensor' type='contact'>
                 <always_on>true</always_on>
                 <update_rate>100</update_rate>
@@ -266,10 +298,11 @@
                     <bumperTopicName>${name}_pinky_medial_bumper</bumperTopicName>
                 </plugin>
-            </sensor>
-            <material>DLR/LightGrey</material>
+            </sensor> -->
+            <material>DLR/LightGrey</material>
+            <xacro:insert_block name="gazebo_friction_properties"/>
         </gazebo>
         <gazebo reference="${name}_pinky_distal_link">
-            <selfCollide>true</selfCollide>
-            <sensor name='${name}_pinky_distal_contact_sensor' type='contact'>
+            <!-- <selfCollide>true</selfCollide>  -->
+            <!-- <sensor name='${name}_pinky_distal_contact_sensor' type='contact'>
                 <always_on>true</always_on>
                 <update_rate>100</update_rate>
@@ -283,6 +316,7 @@
                     <bumperTopicName>${name}_pinky_distal_bumper</bumperTopicName>
                 </plugin>
-            </sensor>
-            <material>DLR/LightGrey</material>
+            </sensor> -->
+            <material>DLR/LightGrey</material>
+            <xacro:insert_block name="gazebo_friction_properties"/>
         </gazebo>
         <gazebo>

File: dlr_description/urdf/hit2/hit2.inertia.xacro (robot description, xacro)
@@ -12,5 +12,5 @@
     <xacro:property name="gr_to_Kg" value="0.001"/>
     <!-- not so negligible, otherwise simulation fails -->
-    <xacro:property name="negligible_mass" value="${200*gr_to_Kg}"/>
+    <xacro:property name="negligible_mass" value="${1000*gr_to_Kg}"/>
     <xacro:property name="negligible_inertia">
         <origin xyz="0 0 0"/>

File: dlr_description/urdf/hit2/hit2.transmission.xacro (robot description, xacro)
@@ -1,48 +1,48 @@
 <?xml version="1.0"?>
 <robot name="robot" xmlns:xacro="http://www.ros.org/wiki/xacro">
-    <xacro:macro name="dlr_hit2_finger_transmission" params="name">
+    <xacro:macro name="dlr_hit2_finger_transmission" params="name finger_name">
 		<xacro:property name="Interface10" value="hardware_interface/PositionJointInterface"/>
 		<xacro:property name="Interface30" value="hardware_interface/EffortJointInterface"/>
-		<transmission name="${name}_abd_trans">
+		<transmission name="${name}_${finger_name}_abd_trans">
 			<robotNamespace>${name}</robotNamespace>
 			<type>transmission_interface/SimpleTransmission</type>
-			<joint name="${name}_abd_joint">
+			<joint name="${name}_${finger_name}_abd_joint">
 				<hardwareInterface>${Interface10}</hardwareInterface>
 				<!-- <hardwareInterface>${Interface30}</hardwareInterface> -->
 			</joint>
-			<actuator name="${name}_abd_motor">
+			<actuator name="${name}_${finger_name}_abd_motor">
 				<mechanicalReduction>1.0</mechanicalReduction>
 			</actuator>
 		</transmission>
-		<transmission name="${name}_inner_trans">
+		<transmission name="${name}_${finger_name}_inner_trans">
 			<robotNamespace>${name}</robotNamespace>
 			<type>transmission_interface/SimpleTransmission</type>
-			<joint name="${name}_inner_joint">
+			<joint name="${name}_${finger_name}_inner_joint">
 				<hardwareInterface>${Interface10}</hardwareInterface>
 				<!-- <hardwareInterface>${Interface30}</hardwareInterface> -->
 			</joint>
-			<actuator name="${name}_inner_motor">
+			<actuator name="${name}_${finger_name}_inner_motor">
 				<mechanicalReduction>1.0</mechanicalReduction>
 			</actuator>
 		</transmission>
-		<transmission name="${name}_outer1_trans">
+		<transmission name="${name}_${finger_name}_outer1_trans">
 			<robotNamespace>${name}</robotNamespace>
 			<type>transmission_interface/SimpleTransmission</type>
-			<joint name="${name}_outer1_joint">
+			<joint name="${name}_${finger_name}_outer1_joint">
 				<hardwareInterface>${Interface10}</hardwareInterface>
 				<!-- <hardwareInterface>${Interface30}</hardwareInterface> -->
 			</joint>
-			<actuator name="${name}_outer1_motor">
+			<actuator name="${name}_${finger_name}_outer1_motor">
 				<mechanicalReduction>1.0</mechanicalReduction>
 			</actuator>
 		</transmission>
-		<transmission name="${name}_outer2_trans">
+		<transmission name="${name}_${finger_name}_outer2_trans">
 			<robotNamespace>${name}</robotNamespace>
 			<type>transmission_interface/SimpleTransmission</type>
-			<joint name="${name}_outer2_joint">
+			<joint name="${name}_${finger_name}_outer2_joint">
 				<hardwareInterface>${Interface10}</hardwareInterface>
 				<!-- <hardwareInterface>${Interface30}</hardwareInterface> -->
 			</joint>
-			<actuator name="${name}_outer2_motor">
+			<actuator name="${name}_${finger_name}_outer2_motor">
 				<mechanicalReduction>1.0</mechanicalReduction>
 			</actuator>
@@ -73,9 +73,9 @@
 	<xacro:macro name="dlr_hit2_transmission" params="name">
 		<!-- five equal fingers -->
-		<xacro:dlr_hit2_finger_transmission name="thumb" />
-		<xacro:dlr_hit2_finger_transmission name="index" />
-		<xacro:dlr_hit2_finger_transmission name="middle" />
-		<xacro:dlr_hit2_finger_transmission name="ring" />
-		<xacro:dlr_hit2_finger_transmission name="pinky" />
+		<xacro:dlr_hit2_finger_transmission name="${name}" finger_name="thumb" />
+		<xacro:dlr_hit2_finger_transmission name="${name}" finger_name="index" />
+		<xacro:dlr_hit2_finger_transmission name="${name}" finger_name="middle" />
+		<xacro:dlr_hit2_finger_transmission name="${name}" finger_name="ring" />
+		<xacro:dlr_hit2_finger_transmission name="${name}" finger_name="pinky" />
 	</xacro:macro>
 </robot>
